Commit message: feat friccion rodillo-carcasa

File: src/omni_description/urdf/mecanum_wheel.xacro (robot description, xacro)
@@ -102,4 +102,5 @@
             <child link="${prefix}_roller_1"/>
             <axis xyz="2.402031829551454e-07 -4.4441721530619205e-07 0.9999998529743616"/>
+            <dynamics damping="0.005" friction="0.001"/>
         </joint>
         <link name="${prefix}_roller_2">
@@ -131,4 +132,5 @@
             <child link="${prefix}_roller_2"/>
             <axis xyz="4.72187707212246e-07 -3.7811381864427673e-07 0.9999999731893168"/>
+            <dynamics damping="0.005" friction="0.001"/>
         </joint>
         <link name="${prefix}_roller_3">
@@ -160,4 +162,5 @@
             <child link="${prefix}_roller_3"/>
             <axis xyz="-3.0094495512278385e-07 1.08901604845002e-07 1.0000003567723852"/>
+            <dynamics damping="0.005" friction="0.001"/>
         </joint>
         <link name="${prefix}_roller_4">
@@ -189,4 +192,5 @@
             <child link="${prefix}_roller_4"/>
             <axis xyz="-4.843221603038905e-07 5.850288692377248e-08 1.0000002354328532"/>
+            <dynamics damping="0.005" friction="0.001"/>
         </joint>
         <link name="${prefix}_roller_5">
@@ -218,4 +222,5 @@
             <child link="${prefix}_roller_5"/>
             <axis xyz="3.458780886145263e-07 3.245384191941092e-07 1.0000002259128622"/>
+            <dynamics damping="0.005" friction="0.001"/>
         </joint>
         <link name="${prefix}_roller_6">
@@ -247,4 +252,5 @@
             <child link="${prefix}_roller_6"/>
             <axis xyz="-4.184712762977938e-07 2.657143597234457e-07 0.999999849860866"/>
+            <dynamics damping="0.005" friction="0.001"/>
         </joint>
         <link name="${prefix}_roller_7">
@@ -276,4 +282,5 @@
             <child link="${prefix}_roller_7"/>
             <axis xyz="1.7805425323036417e-07 -5.224691109750879e-07 1.0000000910443436"/>
+            <dynamics damping="0.005" friction="0.001"/>
         </joint>
         <link name="${prefix}_roller_8">
@@ -305,4 +312,5 @@
             <child link="${prefix}_roller_8"/>
             <axis xyz="1.6116768349061505e-07 -1.155820350540182e-08 1.0000003330324314"/>
+            <dynamics damping="0.005" friction="0.001"/>
         </joint>
         <link name="${prefix}_roller_9">
@@ -334,4 +342,5 @@
             <child link="${prefix}_roller_9"/>
             <axis xyz="-1.5901610209145822e-07 -2.990393351276488e-07 1.0000000674784404"/>
+            <dynamics damping="0.005" friction="0.001"/>
         </joint>
     </xacro:macro>
@@ -424,4 +433,5 @@
             <child link="${prefix}_roller_1"/>
             <axis xyz="-1.780542526197415e-07 -5.224691118077551e-07 1.0000000910443436"/>
+            <dynamics damping="0.005" friction="0.001"/>
         </joint>
         <link name="${prefix}_roller_2">
@@ -453,4 +463,5 @@
             <child link="${prefix}_roller_2"/>
             <axis xyz="4.184712774080168e-07 2.657143595014011e-07 0.9999998498608658"/>
+            <dynamics damping="0.005" friction="0.001"/>
         </joint>
         <link name="${prefix}_roller_3">
@@ -482,4 +493,5 @@
             <child link="${prefix}_roller_3"/>
             <axis xyz="-3.458780878373702e-07 3.245384199712653e-07 1.0000002259128622"/>
+            <dynamics damping="0.005" friction="0.001"/>
         </joint>
         <link name="${prefix}_roller_4">
@@ -511,4 +523,5 @@
             <child link="${prefix}_roller_4"/>
             <axis xyz="4.843221604808323e-07 5.850288786746205e-08 1.0000002354328532"/>
+            <dynamics damping="0.005" friction="0.001"/>
         </joint>
         <link name="${prefix}_roller_5">
@@ -540,4 +553,5 @@
             <child link="${prefix}_roller_5"/>
             <axis xyz="3.009449549284948e-07 1.0890160589971387e-07 1.0000003567723854"/>
+            <dynamics damping="0.005" friction="0.001"/>
         </joint>
         <link name="${prefix}_roller_6">
@@ -569,4 +583,5 @@
             <child link="${prefix}_roller_6"/>
             <axis xyz="-4.721877082669579e-07 -3.7811381814467637e-07 0.9999999731893168"/>
+            <dynamics damping="0.005" friction="0.001"/>
         </joint>
         <link name="${prefix}_roller_7">
@@ -598,4 +613,5 @@
             <child link="${prefix}_roller_7"/>
             <axis xyz="-2.40203183898835e-07 -4.4441721586130356e-07 0.9999998529743617"/>
+            <dynamics damping="0.005" friction="0.001"/>
         </joint>
         <link name="${prefix}_roller_8">
@@ -627,4 +643,5 @@
             <child link="${prefix}_roller_8"/>
             <axis xyz="1.5901610195268034e-07 -2.9903933618236067e-07 1.0000000674784406"/>
+            <dynamics damping="0.005" friction="0.001"/>
         </joint>
         <link name="${prefix}_roller_9">
@@ -656,4 +673,5 @@
             <child link="${prefix}_roller_9"/>
             <axis xyz="-1.6116768346285948e-07 -1.1558204560113694e-08 1.0000003330324314"/>
+            <dynamics damping="0.005" friction="0.001"/>
         </joint>
     </xacro:macro>
