Commit message: borra llantas normales

File: src/omni_description/urdf/omni_urdf.xacro (robot description, xacro)
@@ -6,12 +6,12 @@
         <inertial>
             <origin xyz="0.00498197982182523 5.70233829969297E-05 -0.0121008098068578" rpy="0 0 0"/>
-            <mass value="0.486218814966626"/>
+            <mass value="4.86218814966626"/>
             <inertia
-                    ixx="0.00196277727666921"
-                    ixy="2.50447049446755E-07"
-                    ixz="0.000140534767811098"
-                    iyy="0.00457256033711368"
-                    iyz="2.68618064993882E-07"
-                    izz="0.00493927269870476"/>
+                    ixx="0.196277727666921"
+                    ixy="0.0"
+                    ixz="0.0"
+                    iyy="0.457256033711368"
+                    iyz="0.0"
+                    izz="0.493927269870476"/>
         </inertial>
         <visual>
@@ -36,129 +36,7 @@
         <origin xyz="0.0 0.0 0.0815" rpy="0 0 0"/>
     </joint>
-<!--
-    <link name="front_right_wheel">
-        <inertial>
-            <origin xyz="1.9051E-06 -2.3183E-07 -0.00064079" rpy="0 0 0"/>
-            <mass value="0.051532"/>
-            <inertia ixx="1.4595E-05" ixy="-4.3975E-10" ixz="4.415E-10"
-                     iyy="1.4594E-05" iyz="-1.7476E-09" izz="2.4264E-05"/>
-        </inertial>
-        <visual>
-            <origin xyz="0 0 0" rpy="0 0 0"/>
-            <geometry>
-                <mesh filename="${f_r_wheel}"/>
-            </geometry>
-            <material name="">
-                <color rgba="0.7 0.7 0.7 1"/>
-            </material>
-        </visual>
-        <collision>
-            <origin xyz="0 0 0" rpy="0 0 0"/>
-            <geometry>
-                <mesh filename="${f_r_wheel}"/>
-            </geometry>
-        </collision>
-    </link>
-    <joint name="front_right_joint" type="continuous">
-        <origin xyz="${f_r_wheel_xyz}" rpy="-1.5703 0 3.14159"/>
-        <parent link="base_link"/>
-        <child link="front_right_wheel"/>
-        <axis xyz="0 0 1" rpy="0 0 0"/>
-        <limit effort="100" velocity="25.0"/>
-    </joint>
-    <link name="front_left_wheel">
-        <inertial>
-            <origin xyz="2.3728E-06 -9.4228E-07 0.00064068" rpy="0 0 0"/>
-            <mass value="0.051543"/>
-            <inertia ixx="1.4597E-05" ixy="-4.7945E-10" ixz="-2.4786E-10"
-                     iyy="1.4598E-05" iyz="1.7972E-09" izz="2.4267E-05"/>
-        </inertial>
-        <visual>
-            <origin xyz="0 0 0" rpy="0 0 0"/>
-            <geometry>
-                <mesh filename="${f_l_wheel}"/>
-            </geometry>
-            <material name="">
-                <color rgba="0.7 0.7 0.7 1"/>
-            </material>
-        </visual>
-        <collision>
-            <origin xyz="0 0 0" rpy="0 0 0"/>
-            <geometry>
-                <mesh filename="${f_l_wheel}"/>
-            </geometry>
-        </collision>
-    </link>
-    <joint name="front_left_joint" type="continuous">
-        <origin xyz="${f_l_wheel_xyz}" rpy="1.5703 0 0"/>
-        <parent link="base_link"/>
-        <child link="front_left_wheel"/>
-        <axis xyz="0 0 1" rpy="0 0 0"/>
-        <limit effort="100" velocity="25.0"/>
-    </joint>
-    <link name="back_right_wheel">
-        <inertial>
-            <origin xyz="-1.75924169923403E-06 1.28388821071107E-06 -0.000590549296238266" rpy="0 0 0"/>
-            <mass value="0.051540174053366"/>
-            <inertia ixx="1.45974152250002E-05" ixy="1.94850559178397E-10" ixz="-1.61846387282284E-09"
-                     iyy="1.4596501955693E-05" iyz="-6.27904057423818E-10" izz="2.42663091380451E-05"/>
-        </inertial>
-        <visual>
-            <origin xyz="0 0 0" rpy="0 0 0"/>
-            <geometry>
-                <mesh filename="${b_r_wheel}"/>
-            </geometry>
-            <material name="">
-                <color rgba="0.7 0.7 0.7 1"/>
-            </material>
-        </visual>
-        <collision>
-            <origin xyz="0 0 0" rpy="0 0 0"/>
-            <geometry>
-                <mesh filename="${b_r_wheel}"/>
-            </geometry>
-        </collision>
-    </link>
-    <joint name="back_right_joint" type="continuous">
-        <origin xyz="${b_r_wheel_xyz}" rpy="-1.57 0 3.14159"/>
-        <parent link="base_link"/>
-        <child link="back_right_wheel"/>
-        <axis xyz="0 0 1" rpy="0 0 0"/>
-        <limit effort="100" velocity="25.0"/>
-    </joint>
-    <link name="back_left_wheel">
-        <inertial>
-            <origin xyz="-4.01213085227115E-07 2.04910264598596E-06 0.000590775697051377" rpy="0 0 0"/>
-            <mass value="0.0515309299357028"/>
-            <inertia ixx="1.45942986129926E-05" ixy="-3.19787215398093E-10" ixz="1.74943062058915E-09"
-                     iyy="1.45948727598913E-05" iyz="1.61769812110049E-10" izz="2.4263683888153E-05"/>
-        </inertial>
-        <visual>
-            <origin xyz="0 0 0" rpy="0 0 0"/>
-            <geometry>
-                <mesh filename="${b_l_wheel}"/>
-            </geometry>
-            <material name="">
-                <color rgba="0.7 0.7 0.7 1"/>
-            </material>
-        </visual>
-        <collision>
-            <origin xyz="0 0 0" rpy="0 0 0"/>
-            <geometry>
-                <mesh filename="${b_l_wheel}"/>
-            </geometry>
-        </collision>
-    </link>
-    <joint name="back_left_joint" type="continuous">
-        <origin xyz="${b_l_wheel_xyz}" rpy="1.5703 0 0"/>
-        <parent link="base_link"/>
-        <child link="back_left_wheel"/>
-        <axis xyz="0 0 1" rpy="0 0 0"/>
-        <limit effort="100" velocity="25.0"/>
-    </joint>
--->
-<!-- Ruedas mecanum propias.
-         X: FL y BR llevan la misma quiralidad (derecha), FR y BL la otra (izquierda).
-         Las posiciones/orientaciones son las mismas que usaba la rueda anterior. -->
+<!-- Ruedas mecanum.
+        X: FL y BR llevan la misma quiralidad (derecha), FR y BL la otra (izquierda).
+        Las posiciones/orientaciones son las mismas que usaba la rueda anterior. -->
     <xacro:mecanum_wheel_derecha   prefix="front_left"  parent="base_link" xyz="${f_l_wheel_xyz}" rpy="1.5703 0 0"/>
     <xacro:mecanum_wheel_izquierda prefix="front_right" parent="base_link" xyz="${f_r_wheel_xyz}" rpy="-1.5703 0 3.14159"/>

Commit message: feat: Aumenta masa de robot

File: src/omni_description/urdf/omni_urdf.xacro (robot description, xacro)
@@ -6,5 +6,5 @@
         <inertial>
             <origin xyz="0.00498197982182523 5.70233829969297E-05 -0.0121008098068578" rpy="0 0 0"/>
-            <mass value="4.86218814966626"/>
+            <mass value="5.0"/>
             <inertia
                     ixx="0.196277727666921"
