Commit message: Lidar, DofbotCamera, DepthCamera activos en Gacebo

File: src/dofbot_description/urdf/monocular_camera_sensor.xacro (robot description, xacro)
@@ -39,11 +39,11 @@
   <!-- MONOCULAR CAMERA -->
   <gazebo reference="monocular_camera_link">
-    <material>Gazebo/Orange</material>
-    <sensor type="camera" name="camera">
+    <sensor type="camera" name="mono_camera">
       <always_on>true</always_on>
       <update_rate>30.0</update_rate>
-      <visualize>true</visualize>
+      <topic>mono_camera/image_raw</topic>
+      <gz_frame_id>monocular_camera_link</gz_frame_id>
       <camera>
-        <horizontal_fov>1.085595</horizontal_fov>
+        <horizontal_fov>0.7142</horizontal_fov>
         <image>
           <width>640</width>
@@ -55,23 +55,5 @@
           <far>8.0</far>
         </clip>
-        <distortion>
-         <k1>0.0</k1>
-         <k2>0.0</k2>
-         <k3>0.0</k3>
-         <p1>0.0</p1>
-         <p2>0.0</p2>
-         <center>0.5 0.5</center>
-       </distortion>
       </camera>
-        <plugin name="monocular_camera_plugin" filename="libgazebo_ros_camera.so">
-            <ros>
-                <!--namespace>/</namespace-->
-                <remapping>~/image_raw:=/mono_camera/image_raw</remapping>
-                <remapping>~/camera_info:=/mono_camera/camera_info</remapping>
-            </ros>
-            <camera_name>mono_camera</camera_name>
-            <frame_name>monocular_camera_link</frame_name>
-            <hack_baseline>0.2</hack_baseline>
-        </plugin>
     </sensor>
   </gazebo>

File: src/omni_description/urdf/camera_sensor.xacro (robot description, xacro)
@@ -37,8 +37,9 @@
   </joint>
   <gazebo reference="camera_link">
-    <sensor type="depth" name="camera">
+    <sensor type="rgbd_camera" name="camera">
       <always_on>true</always_on>
       <update_rate>30.0</update_rate>
-      <visualize>true</visualize>
+      <topic>camera</topic>
+      <gz_frame_id>camera_link</gz_frame_id>
       <camera>
         <horizontal_fov>1.085595</horizontal_fov>
@@ -52,23 +53,11 @@
           <far>8.0</far>
         </clip>
-        <distortion>
-         <k1>0.0</k1>
-         <k2>0.0</k2>
-         <k3>0.0</k3>
-         <p1>0.0</p1>
-         <p2>0.0</p2>
-         <center>0.5 0.5</center>
-       </distortion>
+        <depth_camera>
+          <clip>
+            <near>0.1</near>
+            <far>8.0</far>
+          </clip>
+        </depth_camera>
       </camera>
-        <plugin name="camera_plugin" filename="libgazebo_ros_camera.so">
-            <ros>
-                <!--namespace>/</namespace-->
-                <remapping>~/image_raw:=image_raw</remapping>
-                <remapping>~/camera_info:=camera_info</remapping>
-            </ros>
-            <camera_name>camera</camera_name>
-            <frame_name>camera_PC_link</frame_name>
-            <hack_baseline>0.2</hack_baseline>
-        </plugin>
     </sensor>
   </gazebo>

File: src/omni_description/urdf/imu_sensor.xacro (robot description, xacro)
@@ -9,67 +9,62 @@
     <gazebo reference="imu_link">
         <sensor name="imu" type="imu">
-        <visualize>true</visualize>
-        <always_on>true</always_on>
-        <update_rate>30</update_rate>
-        <plugin name="imu_plugin" filename="libgazebo_ros_imu_sensor.so">
-            <ros>
-                <remapping>~/out:=imu</remapping>
-            </ros>
-            <initial_orientation_as_reference>false</initial_orientation_as_reference>
-        </plugin>
-        <imu>
-            <angular_velocity>
-            <x>
-                <noise type="gaussian">
-                <mean>0.0</mean>
-                <stddev>2e-4</stddev>
-                <bias_mean>0.0000075</bias_mean>
-                <bias_stddev>0.0000008</bias_stddev>
-                </noise>
-            </x>
-            <y>
-                <noise type="gaussian">
-                <mean>0.0</mean>
-                <stddev>2e-4</stddev>
-                <bias_mean>0.0000075</bias_mean>
-                <bias_stddev>0.0000008</bias_stddev>
-                </noise>
-            </y>
-            <z>
-                <noise type="gaussian">
-                <mean>0.0</mean>
-                <stddev>2e-4</stddev>
-                <bias_mean>0.0000075</bias_mean>
-                <bias_stddev>0.0000008</bias_stddev>
-                </noise>
-            </z>
-            </angular_velocity>
-            <linear_acceleration>
-            <x>
-                <noise type="gaussian">
-                <mean>0.0</mean>
-                <stddev>1.7e-2</stddev>
-                <bias_mean>0.1</bias_mean>
-                <bias_stddev>0.001</bias_stddev>
-                </noise>
-            </x>
-            <y>
-                <noise type="gaussian">
-                <mean>0.0</mean>
-                <stddev>1.7e-2</stddev>
-                <bias_mean>0.1</bias_mean>
-                <bias_stddev>0.001</bias_stddev>
-                </noise>
-            </y>
-            <z>
-                <noise type="gaussian">
-                <mean>0.0</mean>
-                <stddev>1.7e-2</stddev>
-                <bias_mean>0.1</bias_mean>
-                <bias_stddev>0.001</bias_stddev>
-                </noise>
-            </z>
-            </linear_acceleration>
-        </imu>
+            <always_on>true</always_on>
+            <update_rate>30</update_rate>
+            <topic>imu</topic>
+            <gz_frame_id>imu_link</gz_frame_id>
+            <imu>
+                <angular_velocity>
+                    <x>
+                        <noise type="gaussian">
+                            <mean>0.0</mean>
+                            <stddev>2e-4</stddev>
+                            <bias_mean>0.0000075</bias_mean>
+                            <bias_stddev>0.0000008</bias_stddev>
+                        </noise>
+                    </x>
+                    <y>
+                        <noise type="gaussian">
+                            <mean>0.0</mean>
+                            <stddev>2e-4</stddev>
+                            <bias_mean>0.0000075</bias_mean>
+                            <bias_stddev>0.0000008</bias_stddev>
+                        </noise>
+                    </y>
+                    <z>
+                        <noise type="gaussian">
+                            <mean>0.0</mean>
+                            <stddev>2e-4</stddev>
+                            <bias_mean>0.0000075</bias_mean>
+                            <bias_stddev>0.0000008</bias_stddev>
+                        </noise>
+                    </z>
+                </angular_velocity>
+                <linear_acceleration>
+                    <x>
+                        <noise type="gaussian">
+                            <mean>0.0</mean>
+                            <stddev>1.7e-2</stddev>
+                            <bias_mean>0.1</bias_mean>
+                            <bias_stddev>0.001</bias_stddev>
+                        </noise>
+                    </x>
+                    <y>
+                        <noise type="gaussian">
+                            <mean>0.0</mean>
+                            <stddev>1.7e-2</stddev>
+                            <bias_mean>0.1</bias_mean>
+                            <bias_stddev>0.001</bias_stddev>
+                        </noise>
+                    </y>
+                    <z>
+                        <noise type="gaussian">
+                            <mean>0.0</mean>
+                            <stddev>1.7e-2</stddev>
+                            <bias_mean>0.1</bias_mean>
+                            <bias_stddev>0.001</bias_stddev>
+                        </noise>
+                    </z>
+                </linear_acceleration>
+            </imu>
         </sensor>
     </gazebo>

File: src/omni_description/urdf/lidar_sensor.xacro (robot description, xacro)
@@ -31,21 +31,28 @@
     </joint>
   <gazebo reference="laser_link">
-    <sensor type="ray" name="lidar">
+    <sensor type="gpu_lidar" name="lidar">
       <pose>0 0 0 0 0 0</pose>
       <visualize>$(arg laser_visual)</visualize>
       <always_on>true</always_on>
-      <update_rate>15</update_rate>
-      <ray>
+      <update_rate>12</update_rate>
+      <topic>scan</topic>
+      <gz_frame_id>laser_link</gz_frame_id>
+      <lidar>
         <scan>
           <horizontal>
-            <samples>360</samples>
+            <samples>1667</samples>
             <resolution>1</resolution>
-            <min_angle>-3.14</min_angle>
-            <max_angle>3.14</max_angle>
+            <min_angle>-3.141593</min_angle>
+            <max_angle>3.137823</max_angle>
           </horizontal>
+          <vertical>
+            <samples>1</samples>
+            <min_angle>0</min_angle>
+            <max_angle>0</max_angle>
+          </vertical>
         </scan>
         <range>
-          <min>0.15</min>
-          <max>1.5</max>
+          <min>0.05</min>
+          <max>30.0</max>
           <resolution>0.017453</resolution>
         </range>
@@ -55,16 +62,6 @@
           <stddev>0.01</stddev>
         </noise>
-      </ray>
-      <plugin name="laser_plugin" filename="libgazebo_ros_ray_sensor.so">
-        <ros>
-            <remapping>~/out:=scan</remapping>
-        </ros>
-        <output_type>sensor_msgs/LaserScan</output_type>
-        <frame_name>laser_link</frame_name>
-      </plugin>
+      </lidar>
     </sensor>
   </gazebo>
-      <gazebo reference="laser_link" >
-        <material>Gazebo/Grey</material>
-    </gazebo>
 </robot>

File: src/omni_dofbot_description/urdf/omni_dofbot_urdf.xacro (robot description, xacro)
@@ -6,11 +6,11 @@
   <xacro:include filename="$(find omni_dofbot_description)/urdf/dofbot_without_base_urdf.xacro" />-->
   <xacro:include filename="$(find dofbot_description)/urdf/dofbot_arm_urdf.xacro" />
+  <xacro:include filename="$(find omni_description)/urdf/lidar_sensor.xacro" />
+  <xacro:include filename="$(find omni_description)/urdf/camera_sensor.xacro" />
+  <xacro:include filename="$(find dofbot_description)/urdf/monocular_camera_sensor.xacro"/>
   <!-- Sensores todavía no actualizados para gazebo harmonic, se mantienen los originales de Gazebo Classic para futuras actualizaciones -->
    <!--
    <xacro:include filename="$(find dofbot_description)/urdf/dofbot_sensors_urdf.xacro" />
-  <xacro:include filename="$(find omni_description)/urdf/camera_sensor.xacro" />
-  <xacro:include filename="$(find omni_description)/urdf/lidar_sensor.xacro" />
-  <xacro:include filename="$(find dofbot_description)/urdf/monocular_camera_sensor.xacro"/>
-  <xacro:include filename="$(find omni_description)/urdf/imu_sensor.xacro"/>
+   <xacro:include filename="$(find omni_description)/urdf/imu_sensor.xacro"/>
    -->
   <joint name="omni_to_dofbot_joint" type="fixed">
